Commit message: Add compliance environment and change collisions to stl-files

File: franka_description/urdf/panda_arm.xacro (robot description, xacro)
@@ -45,19 +45,6 @@
       </visual>
       <collision>
-        <origin xyz="-0.075 0 0.06" rpy="0 ${pi/2} 0" />
-        <geometry>
-          <cylinder radius="${0.06+safety_distance}" length="0.03" />
-        </geometry>
-      </collision>
-      <collision>
-        <origin xyz="-0.06 0 0.06" rpy="0 0 0" />
-        <geometry>
-          <sphere radius="${0.06+safety_distance}" />
-        </geometry>
-      </collision>
-      <collision>
-        <origin xyz="-0.09 0 0.06" rpy="0 0 0" />
-        <geometry>
-          <sphere radius="${0.06+safety_distance}" />
+        <geometry>
+          <mesh filename="file://$(find ${description_pkg})/meshes/collision/link0.stl" />
         </geometry>
       </collision>
@@ -70,19 +57,6 @@
       </visual>
       <collision>
-        <origin xyz="0 0 -0.1915" rpy="0 0 0" />
-        <geometry>
-          <cylinder radius="${0.06+safety_distance}" length="0.2830" />
-        </geometry>
-      </collision>
-      <collision>
-        <origin xyz="0 0 -0.333" rpy="0 0 0" />
-        <geometry>
-          <sphere radius="${0.06+safety_distance}" />
-        </geometry>
-      </collision>
-      <collision>
-        <origin xyz="0 0 -0.05" rpy="0 0 0" />
-        <geometry>
-          <sphere radius="${0.06+safety_distance}" />
+        <geometry>
+          <mesh filename="file://$(find ${description_pkg})/meshes/collision/link1.stl" />
         </geometry>
       </collision>
@@ -108,19 +82,6 @@
       </visual>
       <collision>
-        <origin xyz="0 0 0" rpy="0 0 0" />
-        <geometry>
-          <cylinder radius="${0.06+safety_distance}" length="0.12" />
-        </geometry>
-      </collision>
-      <collision>
-        <origin xyz="0 0 -0.06" rpy="0 0 0" />
-        <geometry>
-          <sphere radius="${0.06+safety_distance}" />
-        </geometry>
-      </collision>
-      <collision>
-        <origin xyz="0 0 0.06" rpy="0 0 0" />
-        <geometry>
-          <sphere radius="${0.06+safety_distance}" />
+        <geometry>
+          <mesh filename="file://$(find ${description_pkg})/meshes/collision/link2.stl" />
         </geometry>
       </collision>
@@ -146,19 +107,6 @@
       </visual>
       <collision>
-        <origin xyz="0 0 -0.145" rpy="0 0 0" />
-        <geometry>
-          <cylinder radius="${0.06+safety_distance}" length="0.15" />
-        </geometry>
-      </collision>
-      <collision>
-        <origin xyz="0 0 -0.22" rpy="0 0 0" />
-        <geometry>
-          <sphere radius="${0.06+safety_distance}" />
-        </geometry>
-      </collision>
-      <collision>
-        <origin xyz="0 0 -0.07" rpy="0 0 0" />
-        <geometry>
-          <sphere radius="${0.06+safety_distance}" />
+        <geometry>
+          <mesh filename="file://$(find ${description_pkg})/meshes/collision/link3.stl" />
         </geometry>
       </collision>
@@ -184,19 +132,6 @@
       </visual>
       <collision>
-        <origin xyz="0 0 0" rpy="0 0 0" />
-        <geometry>
-          <cylinder radius="${0.06+safety_distance}" length="0.12" />
-        </geometry>
-      </collision>
-      <collision>
-        <origin xyz="0 0 0.06" rpy="0 0 0" />
-        <geometry>
-          <sphere radius="${0.06+safety_distance}" />
-        </geometry>
-      </collision>
-      <collision>
-        <origin xyz="0 0 -0.06" rpy="0 0 0" />
-        <geometry>
-          <sphere radius="${0.06+safety_distance}" />
+        <geometry>
+          <mesh filename="file://$(find ${description_pkg})/meshes/collision/link4.stl" />
         </geometry>
       </collision>
@@ -222,37 +157,6 @@
       </visual>
       <collision>
-        <origin xyz="0 0 -0.26" rpy="0 0 0" />
-        <geometry>
-          <cylinder radius="${0.06+safety_distance}" length="0.1" />
-        </geometry>
-      </collision>
-      <collision>
-        <origin xyz="0 0 -0.31" rpy="0 0 0" />
-        <geometry>
-          <sphere radius="${0.06+safety_distance}" />
-        </geometry>
-      </collision>
-      <collision>
-        <origin xyz="0 0 -0.21" rpy="0 0 0" />
-        <geometry>
-          <sphere radius="${0.06+safety_distance}" />
-        </geometry>
-      </collision>
-      <collision>
-        <origin xyz="0 0.08 -0.13" rpy="0 0 0" />
-        <geometry>
-          <cylinder radius="${0.025+safety_distance}" length="0.14" />
-        </geometry>
-      </collision>
-      <collision>
-        <origin xyz="0 0.08 -0.06" rpy="0 0 0" />
-        <geometry>
-          <sphere radius="${0.025+safety_distance}" />
-        </geometry>
-      </collision>
-      <collision>
-        <origin xyz="0 0.08 -0.20" rpy="0 0 0" />
-        <geometry>
-          <sphere radius="${0.025+safety_distance}" />
+        <geometry>
+          <mesh filename="file://$(find ${description_pkg})/meshes/collision/link5.stl" />
         </geometry>
       </collision>
@@ -278,19 +182,6 @@
       </visual>
       <collision>
-        <origin xyz="0 0 -0.03" rpy="0 0 0" />
-        <geometry>
-          <cylinder radius="${0.05+safety_distance}" length="0.08" />
-        </geometry>
-      </collision>
-      <collision>
-        <origin xyz="0 0 0.01" rpy="0 0 0" />
-        <geometry>
-          <sphere radius="${0.05+safety_distance}" />
-        </geometry>
-      </collision>
-      <collision>
-        <origin xyz="0 0 -0.07" rpy="0 0 0" />
-        <geometry>
-          <sphere radius="${0.05+safety_distance}" />
+        <geometry>
+          <mesh filename="file://$(find ${description_pkg})/meshes/collision/link6.stl" />
         </geometry>
       </collision>
@@ -316,19 +207,6 @@
       </visual>
       <collision>
-        <origin xyz="0 0 0.01" rpy="0 0 0" />
-        <geometry>
-          <cylinder radius="${0.04+safety_distance}" length="0.14" />
-        </geometry>
-      </collision>
-      <collision>
-        <origin xyz="0 0 0.08" rpy="0 0 0" />
-        <geometry>
-          <sphere radius="${0.04+safety_distance}" />
-        </geometry>
-      </collision>
-      <collision>
-        <origin xyz="0 0 -0.06" rpy="0 0 0" />
-        <geometry>
-          <sphere radius="${0.04+safety_distance}" />
+        <geometry>
+          <mesh filename="file://$(find ${description_pkg})/meshes/collision/link7.stl" />
         </geometry>
       </collision>
