Commit message: Fix computed torque controller input, manipulator base visuals and changed compliance enviroment controller

File: franka_description/urdf/effort_panda_arm_ft_sensor.urdf.xacro (robot description, xacro)
@@ -28,5 +28,5 @@
       <origin xyz="0 0 0.5" rpy="0 0 0" />
       <geometry>
-        <box size="1.7 0.5 1" />
+        <box size="1.71 0.51 1" />
       </geometry>
       <material name="metal">
@@ -37,5 +37,5 @@
       <origin xyz="0 0 0.5" rpy="0 0 0" />
       <geometry>
-        <box size="1.7 0.5 1" />
+        <box size="1.71 0.51 1" />
       </geometry>
     </collision>
