Commit message: updated changes

File: franka_description/urdf/effort_panda_arm_cam.urdf.xacro (robot description, xacro)
@@ -57,6 +57,22 @@
       safety_distance="0.03" />
   </xacro:if>
+  <xacro:if value="$(arg hand)">
+	<xacro:include filename="$(find franka_description)/urdf/rgb_camera.xacro"/>
+	<!-- where you define the robot links -->
+	<xacro:rgb_camera
+	  parent_link="panda_link7"
+	  camera_name="wrist_cam"
+	  camera_link_name="camera_link"
+	  camera_optical_link_name="camera_link_optical"
+	  xyz="0 0 0.08" rpy="0 0 0"
+	  width="640" height="480"
+	  hfov="1.047"
+	  update_rate="30"
+	  clip_near="0.05" clip_far="10.0"
+	  topic="/wrist_cam"
+	  visualize="true"/>
+ </xacro:if>
   <xacro:include
-    filename="$(find franka_description)/urdf/ros2_control/panda_arm.ros2_control.xacro" />
+    filename="$(find franka_description)/urdf/ros2_control/effort_panda_arm.ros2_control.xacro" />
   <xacro:panda_arm_ros2_control
     ns="$(arg arm_id)"

File: franka_description/urdf/hand.xacro (robot description, xacro)
@@ -61,4 +61,9 @@
     </joint>
     <link name="${ns}_leftfinger">
+     <inertial>
+       <mass value="0.05"/>
+       <origin xyz="0 0 0" rpy="0 0 0"/>
+       <inertia ixx="1e-5" iyy="1e-5" izz="1e-5" ixy="0" ixz="0" iyz="0"/>
+     </inertial>
       <visual>
         <geometry>
@@ -68,4 +73,9 @@
     </link>
     <link name="${ns}_rightfinger">
+     <inertial>
+       <mass value="0.05"/>
+       <origin xyz="0 0 0" rpy="0 0 0"/>
+       <inertia ixx="1e-5" iyy="1e-5" izz="1e-5" ixy="0" ixz="0" iyz="0"/>
+     </inertial>
       <visual>
         <origin xyz="0 0 0" rpy="0 0 ${pi}"/>
